Commit message: progress

File: src/ROS/create_autonomy/ca_description/urdf/create_wheel.xacro (robot description, xacro)
@@ -5,5 +5,5 @@
   <xacro:property name="parent_link" value="${parent}"/>
   <xacro:property name="link_name"   value="${name}_link"/>
-  <xacro:property name="mass"        value="0.5"/>
+  <xacro:property name="mass"        value="1"/>
   <joint name="${name}_joint" type="continuous">
     <xacro:insert_block name="origin"/>
@@ -27,8 +27,8 @@
   </link>
   <gazebo reference="${link_name}">
-    <mu1>1.0</mu1>
-    <mu2>1.0</mu2>
-    <kp>1000000.0</kp>
-    <kd>100.0</kd>
+    <mu1>10000.0</mu1>
+    <mu2>10000.0</mu2>
+    <kp>100000000.0</kp>
+    <kd>10000.0</kd>
     <minDepth>0.001</minDepth>
     <maxVel>1.0</maxVel>
