Commit message: rosbag done the right way, fix meshes, address visibility taking too long

File: src/ROS/create_autonomy/ca_description/urdf/sensors/lasers/rplidar.xacro (robot description, xacro)
@@ -8,5 +8,5 @@
 <xacro:property name="rate_hz"       value="10"/>
 <xacro:property name="min_range_m"   value="0.15"/>
-<xacro:property name="max_range_m"   value="12.0"/>
+<xacro:property name="max_range_m"   value="15.0"/>
 <xacro:property name="samples"       value="720"/>
 <xacro:property name="resolution_mm" value="0.5"/>
